File: Tag Tracker_v1.brd (EAGLE design)
At the start: 45.5 x 38.4 mm, 69 parts, among them Q1 MMBT2222A, Q2 MMBT2222A, Q3 BSS138, Q4 BSS138, Q5 BSS138, U1 ATMEGA328P_TQFP, U2 FDC6330L, U3 FDC6330L, U4 FDC6330L, U5 FDC6330L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

Commit message: Add files via upload
Parts:
- moved R17 2.22 mm to (32.5, 33.3), turned to 180 degrees
- moved U6 1.82 mm to (21.2, 34.2)
- moved C8 1.79 mm to (21.2, 37.5)
- moved C9 1.44 mm to (24.0, 36.7)
- moved C12 0.68 mm to (37.7, 36.1)
- moved JP2 0.52 mm to (29.7, 35.9)
- moved R10 0.38 mm to (21.2, 35.2)
- moved C13 0.36 mm to (23.5, 34.8)
- moved C16 0.28 mm to (23.5, 33.5)
- moved U$1 0.20 mm to (17.3, 35.1)
Routing:
- net VBAT: track 30.8 -> 93.1 mm, vias 0 -> 6
- net SDA: track 0.00 -> 21.8 mm, vias 0 -> 2
- net SCL: track 0.00 -> 18.6 mm, vias 0 -> 2
- net CNFG: track 0.00 -> 12.0 mm, vias 0 -> 1
- net INT_ACC: track 0.00 -> 11.4 mm
- net 2.8V: track 0.00 -> 10.6 mm
- net MISO: track 12.3 -> 21.3 mm
- net GND: track 22.0 -> 30.7 mm
- net N$46: track 0.00 -> 8.18 mm
- net TXD: track 60.0 -> 67.7 mm, vias 2 -> 3
- net RESET: track 7.51 -> 14.1 mm, vias 0 -> 1
- net SCK: track 13.7 -> 19.2 mm, vias 2 -> 1
- net N$22: track 0.00 -> 3.53 mm
- net N$30: track 0.00 -> 1.85 mm
- net N$14: track 0.00 -> 1.74 mm
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- added copper zone on layer 1, net VBAT
- added copper zone on layer 16, net VBAT

Commit message: Add files via upload
Parts:
- moved C3 1.44 mm to (19.8, 36.6)
- moved R10 0.17 mm to (21.3, 35.3)
Connections:
- net GPS_GAT: no longer U4.P$5, U5.P$5
- net SIM900_GAT: now also U4.P$5, U5.P$5
Routing:
- net GSM_GND: track 0.00 -> 30.1 mm
- net 2.8V: track 10.6 -> 39.1 mm, vias 0 -> 1
- net SIM900_GAT: track 0.00 -> 21.7 mm
- net GPS_VCC: track 1.27 -> 20.1 mm
- net GSM_VCC: track 0.00 -> 18.0 mm, vias 0 -> 2
- net GPS_GAT: track 0.00 -> 13.1 mm
- net NETLIGHT: track 0.00 -> 11.7 mm, vias 0 -> 1
- net N$22: track 3.53 -> 14.7 mm
- net N$18: track 0.00 -> 9.34 mm, vias 0 -> 2
- net GPS_GND: track 1.27 -> 10.2 mm
- net N$27: track 0.00 -> 8.40 mm
- net N$16: track 0.00 -> 7.45 mm
- net GND: track 30.7 -> 37.4 mm
- net N$40: track 0.00 -> 4.79 mm
- net N$48: track 0.00 -> 3.19 mm
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Other:
- board text added: "TO DO: Check SIM header connections!!!"

Commit message: Add files via upload
Parts:
- removed U$2: NANOSIM, myLibraries:NANOSIM
- added U10: NANOSIM, myLibraries:NANOSIM
- moved R7 8.18 mm to (36.1, 16.0)
- moved C5 8.00 mm to (43.9, 16.0)
- moved R5 2.21 mm to (38.2, 16.0)
- moved R1 1.28 mm to (39.6, 16.0)
- moved D2 1.02 mm to (7.62, 35.3)
- moved C1 0.92 mm to (24.3, 17.1)
- moved C7 0.92 mm to (24.3, 18.3)
- moved C10 0.63 mm to (9.91, 35.9)
- moved C2 0.24 mm to (42.1, 16.0)
- moved D3 0.13 mm to (13.2, 36.2)
- moved D1 0.13 mm to (11.9, 36.2)
- renumbered JP9 to MICRO_USB, U$1 to U11, U$5 to U12
Connections:
- net GND: now also U10.C5; no longer U$2.C7
- net N$1: now also U10.C7; no longer U$2.C5
- net N$3: now also R1.1, U10.C2; no longer R5.1, U$2.C1
- net N$7: now also R5.1, U10.C3; no longer R1.1, U$2.C6
- net SIM_VDD: now also U10.C1; no longer U$2.C3
Routing:
- net GND: track 37.4 -> 113.9 mm, vias 1 -> 11
- net SIM900_GAT: track 21.7 -> 54.1 mm, vias 0 -> 2
- net GPS_GAT: track 13.1 -> 43.4 mm, vias 0 -> 2
- net GSM_GND: track 30.1 -> 60.0 mm, vias 0 -> 1
- net GPS_GND: track 10.2 -> 36.0 mm, vias 0 -> 2
- net SIM_VDD: track 14.1 -> 37.4 mm, vias 0 -> 2
- net VBAT: track 91.7 -> 112.8 mm
- net SIM_DATA: track 13.2 -> 30.5 mm
- net DBG: track 0.00 -> 13.7 mm, vias 0 -> 1
- net N$1: track 13.0 -> 23.1 mm
- net SIM_RST: track 11.9 -> 16.2 mm
- net N$13: track 32.7 -> 35.9 mm
- net SIM_CLK: track 13.4 -> 15.7 mm
- net N$18: track 9.34 -> 11.1 mm
- net N$12: track 4.99 -> 6.77 mm
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- added copper zone on layer 16, net GND
- added copper zone on layer 1, net GSM_GND
- added copper zone on layer 16, net N$19
- added copper zone on layer 16, net N$25
Other:
- board text added: "+"
- board text added: "_"
- board text removed: "TO DO: Check SIM header connections!!!"

Commit message: Add files via upload
Parts:
- C14, C15: device SparkFun-Capacitors:0805 -> SparkFun-Capacitors:0603-CAP
- R10: value (none) -> 2K
- moved C15 1.60 mm to (13.5, 19.1)
- moved C14 1.17 mm to (13.5, 17.9)
Routing:
- net GND: track 113.9 -> 110.7 mm
Changed lines of the file:
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@@
 <grid distance="1" unitdist="mil" unit="mil" style="lines" multiple="1" display="yes" altdistance="5" altunitdist="mil" altunit="mil"/>
 <layers>
-<layer number="1" name="Top" color="4" fill="1" visible="yes" active="yes"/>
+<layer number="1" name="Top" color="4" fill="1" visible="no" active="yes"/>
 <layer number="2" name="Route2" color="1" fill="3" visible="no" active="no"/>
 <layer number="3" name="Route3" color="4" fill="3" visible="no" active="no"/>
@@
 <layer number="19" name="Unrouted" color="6" fill="1" visible="yes" active="yes"/>
 <layer number="20" name="Dimension" color="15" fill="1" visible="yes" active="yes"/>
-<layer number="21" name="tPlace" color="7" fill="1" visible="no" active="yes"/>
+<layer number="21" name="tPlace" color="7" fill="1" visible="yes" active="yes"/>
 <layer number="22" name="bPlace" color="7" fill="1" visible="yes" active="yes"/>
 <layer number="23" name="tOrigins" color="15" fill="1" visible="yes" active="yes"/>
 <layer number="24" name="bOrigins" color="15" fill="1" visible="yes" active="yes"/>
-<layer number="25" name="tNames" color="7" fill="1" visible="no" active="yes"/>
+<layer number="25" name="tNames" color="7" fill="1" visible="yes" active="yes"/>
 <layer number="26" name="bNames" color="7" fill="1" visible="yes" active="yes"/>
 <layer number="27" name="tValues" color="7" fill="1" visible="no" active="yes"/>
@@
 <attribute name="NAME" x="40.6146" y="14.4399" size="0.8128" layer="25" font="vector" ratio="10" rot="R180"/>
 </element>
-<element name="R10" library="SparkFun-Resistors" package="0603-RES" value="" x="21.2852" y="35.3314" smashed="yes" rot="MR270">
+<element name="R10" library="SparkFun-Resistors" package="0603-RES" value="2K" x="21.2852" y="35.3314" smashed="yes" rot="MR270">
 <attribute name="NAME" x="21.8821" y="35.4076" size="0.762" layer="26" rot="MR90"/>
 <attribute name="VALUE" x="22.6822" y="36.3474" size="0.4064" layer="28" rot="MR270"/>
@@
 <element name="C6" library="SparkFun-Capacitors" package="1206" value="100uF/6.3V" x="16.129" y="19.05" smashed="yes" rot="MR270">
 <attribute name="NAME" x="17.8308" y="19.6342" size="0.8128" layer="26" font="vector" ratio="10" rot="MR270"/>
-</element>
-<element name="C14" library="SparkFun-Capacitors" package="0805" value="100nF" x="13.462" y="19.05" smashed="yes" rot="MR180">
-<attribute name="NAME" x="8.7376" y="19.2913" size="0.8128" layer="26" font="vector" ratio="10" rot="MR180"/>
-</element>
-<element name="C15" library="SparkFun-Capacitors" package="0805" value="33pF" x="13.462" y="17.526" smashed="yes" rot="MR180">
-<attribute name="NAME" x="8.8646" y="17.9197" size="0.8128" layer="26" font="vector" rot="MR180"/>
 </element>
 <element name="D3" library="led" package="SML0603" value="GREEN (charged)" x="13.208" y="36.195" smashed="yes" rot="MR270">
@@
 <element name="JP2" library="Various_parts" package="TC2030-NL" value="TC2030-NL" x="29.718" y="35.941"/>
 <element name="U10" library="myLibraries" package="NANOSIM" value="NANOSIM" x="40.2844" y="6.4262"/>
+<element name="C15" library="SparkFun-Capacitors" package="0603-CAP" value="33pF" x="13.5128" y="19.1262" smashed="yes" rot="MR180">
+<attribute name="NAME" x="8.6868" y="19.5326" size="0.8128" layer="26" font="vector" ratio="10" rot="MR180"/>
+<attribute name="VALUE" x="12.4968" y="20.2692" size="0.4064" layer="28" font="vector" rot="MR180"/>
+</element>
+<element name="C14" library="SparkFun-Capacitors" package="0603-CAP" value="100nF" x="13.5128" y="17.8816" smashed="yes" rot="MR180">
+<attribute name="NAME" x="8.6868" y="18.2626" size="0.8128" layer="26" font="vector" ratio="10" rot="MR180"/>
+<attribute name="VALUE" x="12.4968" y="19.0246" size="0.4064" layer="28" font="vector" rot="MR180"/>
+</element>
 </elements>
 <signals>
@@
 <wire x1="37.592" y1="32.9376" x2="37.535" y2="32.9946" width="0.2032" layer="16"/>
 <via x="37.084" y="26.035" extent="1-16" drill="0.3048" diameter="0.508"/>
-<contactref element="C14" pad="2"/>
-<contactref element="C15" pad="2"/>
 <contactref element="C6" pad="2"/>
 <contactref element="D3" pad="C"/>
@@
 <wire x1="37.535" y1="35.402" x2="37.535" y2="32.9946" width="0.3048" layer="16"/>
 <wire x1="14.412" y1="20.671" x2="14.412" y2="19.1" width="0.508" layer="16"/>
-<wire x1="14.412" y1="19.1" x2="14.362" y2="19.05" width="0.508" layer="16"/>
-<wire x1="14.362" y1="19.05" x2="14.362" y2="17.526" width="0.508" layer="16"/>
-<wire x1="14.362" y1="17.526" x2="16.005" y2="17.526" width="0.508" layer="16"/>
 <wire x1="16.005" y1="17.526" x2="16.129" y2="17.65" width="0.508" layer="16"/>
 <wire x1="16.129" y1="17.65" x2="18.2596" y2="17.65" width="0.508" layer="16"/>
@@
 <wire x1="13.0302" y1="34.544" x2="13.0556" y2="34.5186" width="0.254" layer="16"/>
 <wire x1="13.0556" y1="34.5186" x2="13.0556" y2="34.4932" width="0.254" layer="16"/>
+<contactref element="C15" pad="2"/>
+<contactref element="C14" pad="2"/>
 </signal>
 <signal name="SIM_DATA">
@@
 <contactref element="U4" pad="P$2"/>
 <contactref element="C6" pad="1"/>
-<contactref element="C15" pad="1"/>
-<contactref element="C14" pad="1"/>
 <contactref element="R15" pad="1"/>
-<wire x1="12.562" y1="17.526" x2="12.562" y2="19.05" width="0.508" layer="16"/>
-<wire x1="12.562" y1="19.05" x2="12.562" y2="20.621" width="0.508" layer="16"/>
 <wire x1="12.562" y1="20.621" x2="12.512" y2="20.671" width="0.4064" layer="16"/>
 <wire x1="9.971" y1="18.97" x2="11.2814" y2="18.97" width="0.508" layer="1"/>
@@
 <wire x1="11.3538" y1="17.6022" x2="10.986" y2="17.97" width="0.508" layer="1"/>
 <via x="11.5062" y="18.669" extent="1-16" drill="0.381" diameter="0.8128"/>
-<wire x1="12.562" y1="17.526" x2="11.5824" y2="17.526" width="0.508" layer="16"/>
 <wire x1="11.5824" y1="17.526" x2="11.5062" y2="17.6022" width="0.508" layer="16"/>
 <wire x1="11.5062" y1="18.669" x2="11.5062" y2="17.6022" width="0.508" layer="16"/>
+<contactref element="C14" pad="1"/>
+<contactref element="C15" pad="1"/>
+<wire x1="12.6628" y1="17.8816" x2="12.6628" y2="19.1262" width="0.4064" layer="16"/>
+<wire x1="12.6628" y1="19.1262" x2="12.2056" y2="18.669" width="0.4064" layer="16"/>
+<wire x1="12.2056" y1="18.669" x2="11.5062" y2="18.669" width="0.4064" layer="16"/>
+<wire x1="12.6628" y1="19.1262" x2="12.512" y2="19.277" width="0.4064" layer="16"/>
+<wire x1="12.512" y1="19.277" x2="12.512" y2="20.671" width="0.4064" layer="16"/>
 </signal>
 <signal name="N$19">
