File: Tag Tracker_v1.sch (EAGLE design)
At the start: 69 parts, among them Q1 MMBT2222A, Q2 MMBT2222A, Q3 BSS138, Q4 BSS138, Q5 BSS138, U1 ATMEGA328P_TQFP, U2 FDC6330L, U3 FDC6330L, U4 FDC6330L, U5 FDC6330L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

Commit message: Add files via upload
Connections:
- net GPS_GAT: no longer U4.O/F, U5.O/F
- net SIM900_GAT: now also U4.O/F, U5.O/F
Other:
- moved on the sheet: R16, R18
Changed lines of the file:
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@@
 <instance part="U4" gate="G$1" x="99.06" y="-81.28"/>
 <instance part="U5" gate="G$1" x="99.06" y="-104.14"/>
-<instance part="R16" gate="G$1" x="121.92" y="-81.134" smashed="yes" rot="R270">
-<attribute name="OC_FARNELL" x="121.92" y="-81.134" size="1.778" layer="96" rot="R270" display="off"/>
-<attribute name="MF" x="121.92" y="-81.134" size="1.778" layer="96" rot="R270" display="off"/>
-<attribute name="MPN" x="121.92" y="-81.134" size="1.778" layer="96" rot="R270" display="off"/>
-<attribute name="NAME" x="117.964" y="-84.0994" size="1.778" layer="95"/>
-<attribute name="VALUE" x="125.222" y="-83.204" size="1.778" layer="96" rot="R90"/>
+<instance part="R16" gate="G$1" x="127" y="-81.134" smashed="yes" rot="R270">
+<attribute name="OC_FARNELL" x="127" y="-81.134" size="1.778" layer="96" rot="R270" display="off"/>
+<attribute name="MF" x="127" y="-81.134" size="1.778" layer="96" rot="R270" display="off"/>
+<attribute name="MPN" x="127" y="-81.134" size="1.778" layer="96" rot="R270" display="off"/>
+<attribute name="NAME" x="123.044" y="-84.0994" size="1.778" layer="95"/>
+<attribute name="VALUE" x="130.302" y="-83.204" size="1.778" layer="96" rot="R90"/>
 </instance>
-<instance part="R18" gate="G$1" x="121.92" y="-104.756" smashed="yes" rot="R270">
-<attribute name="OC_FARNELL" x="121.92" y="-104.756" size="1.778" layer="96" rot="R270" display="off"/>
-<attribute name="MF" x="121.92" y="-104.756" size="1.778" layer="96" rot="R270" display="off"/>
-<attribute name="MPN" x="121.92" y="-104.756" size="1.778" layer="96" rot="R270" display="off"/>
-<attribute name="NAME" x="116.948" y="-108.2294" size="1.778" layer="95"/>
-<attribute name="VALUE" x="125.222" y="-106.826" size="1.778" layer="96" rot="R90"/>
+<instance part="R18" gate="G$1" x="127" y="-104.756" smashed="yes" rot="R270">
+<attribute name="OC_FARNELL" x="127" y="-104.756" size="1.778" layer="96" rot="R270" display="off"/>
+<attribute name="MF" x="127" y="-104.756" size="1.778" layer="96" rot="R270" display="off"/>
+<attribute name="MPN" x="127" y="-104.756" size="1.778" layer="96" rot="R270" display="off"/>
+<attribute name="NAME" x="122.028" y="-108.2294" size="1.778" layer="95"/>
+<attribute name="VALUE" x="130.302" y="-106.826" size="1.778" layer="96" rot="R90"/>
 </instance>
 <instance part="U6" gate="G$1" x="-60.96" y="93.98"/>
@@
 <segment>
 <pinref part="R18" gate="G$1" pin="2"/>
-<wire x1="121.92" y1="-109.836" x2="121.92" y2="-109.22" width="0.1524" layer="91"/>
-<wire x1="121.92" y1="-109.836" x2="121.92" y2="-111.76" width="0.1524" layer="91"/>
+<wire x1="127" y1="-109.836" x2="127" y2="-109.22" width="0.1524" layer="91"/>
+<wire x1="127" y1="-109.836" x2="127" y2="-111.76" width="0.1524" layer="91"/>
 <pinref part="U5" gate="G$1" pin="VIN"/>
-<wire x1="121.92" y1="-111.76" x2="111.76" y2="-111.76" width="0.1524" layer="91"/>
+<wire x1="127" y1="-111.76" x2="111.76" y2="-111.76" width="0.1524" layer="91"/>
 <wire x1="111.76" y1="-111.76" x2="111.76" y2="-106.68" width="0.1524" layer="91"/>
 <label x="114.3" y="-111.76" size="1.778" layer="95"/>
@@
 <segment>
 <pinref part="R16" gate="G$1" pin="2"/>
-<wire x1="121.92" y1="-86.214" x2="121.92" y2="-88.9" width="0.1524" layer="91"/>
+<wire x1="127" y1="-86.214" x2="127" y2="-88.9" width="0.1524" layer="91"/>
 <pinref part="U4" gate="G$1" pin="VIN"/>
-<wire x1="121.92" y1="-88.9" x2="111.76" y2="-88.9" width="0.1524" layer="91"/>
+<wire x1="127" y1="-88.9" x2="111.76" y2="-88.9" width="0.1524" layer="91"/>
 <wire x1="111.76" y1="-88.9" x2="111.76" y2="-83.82" width="0.1524" layer="91"/>
 <label x="114.3" y="-88.9" size="1.778" layer="95"/>
@@
 </segment>
 <segment>
-<pinref part="U4" gate="G$1" pin="O/F"/>
-<wire x1="111.76" y1="-81.28" x2="116.84" y2="-81.28" width="0.1524" layer="91"/>
-<label x="109.22" y="-81.28" size="1.778" layer="95"/>
-</segment>
-<segment>
-<pinref part="U5" gate="G$1" pin="O/F"/>
-<wire x1="111.76" y1="-104.14" x2="116.84" y2="-104.14" width="0.1524" layer="91"/>
-<label x="109.22" y="-104.14" size="1.778" layer="95"/>
-</segment>
-<segment>
 <pinref part="U1" gate="U$1" pin="PD5(T1)"/>
 <wire x1="91.44" y1="48.26" x2="101.6" y2="48.26" width="0.1524" layer="91"/>
@@
 <wire x1="91.44" y1="50.8" x2="101.6" y2="50.8" width="0.1524" layer="91"/>
 <label x="93.98" y="50.8" size="1.778" layer="95"/>
+</segment>
+<segment>
+<pinref part="U4" gate="G$1" pin="O/F"/>
+<wire x1="111.76" y1="-81.28" x2="116.84" y2="-81.28" width="0.1524" layer="91"/>
+<label x="111.76" y="-81.28" size="1.778" layer="95"/>
+</segment>
+<segment>
+<pinref part="U5" gate="G$1" pin="O/F"/>
+<wire x1="111.76" y1="-104.14" x2="116.84" y2="-104.14" width="0.1524" layer="91"/>
+<label x="111.76" y="-104.14" size="1.778" layer="95"/>
 </segment>
 </net>
@@
 <net name="N$30" class="0">
 <segment>
-<wire x1="121.92" y1="-76.454" x2="121.92" y2="-76.054" width="0.1524" layer="91"/>
+<wire x1="127" y1="-76.454" x2="127" y2="-76.054" width="0.1524" layer="91"/>
 <pinref part="U4" gate="G$1" pin="R1C1"/>
-<wire x1="121.92" y1="-76.054" x2="121.92" y2="-73.66" width="0.1524" layer="91"/>
-<wire x1="121.92" y1="-73.66" x2="111.76" y2="-73.66" width="0.1524" layer="91"/>
+<wire x1="127" y1="-76.054" x2="127" y2="-73.66" width="0.1524" layer="91"/>
+<wire x1="127" y1="-73.66" x2="111.76" y2="-73.66" width="0.1524" layer="91"/>
 <wire x1="111.76" y1="-73.66" x2="111.76" y2="-78.74" width="0.1524" layer="91"/>
 <pinref part="R16" gate="G$1" pin="1"/>
-<junction x="121.92" y="-76.054"/>
+<junction x="127" y="-76.054"/>
 </segment>
 </net>
 <net name="N$39" class="0">
 <segment>
-<wire x1="121.92" y1="-99.06" x2="121.92" y2="-99.676" width="0.1524" layer="91"/>
+<wire x1="127" y1="-99.06" x2="127" y2="-99.676" width="0.1524" layer="91"/>
 <pinref part="U5" gate="G$1" pin="R1C1"/>
-<wire x1="121.92" y1="-99.676" x2="121.92" y2="-96.52" width="0.1524" layer="91"/>
-<wire x1="121.92" y1="-96.52" x2="111.76" y2="-96.52" width="0.1524" layer="91"/>
+<wire x1="127" y1="-99.676" x2="127" y2="-96.52" width="0.1524" layer="91"/>
+<wire x1="127" y1="-96.52" x2="111.76" y2="-96.52" width="0.1524" layer="91"/>
 <wire x1="111.76" y1="-96.52" x2="111.76" y2="-101.6" width="0.1524" layer="91"/>
 <pinref part="R18" gate="G$1" pin="1"/>
-<junction x="121.92" y="-99.676"/>
-</segment>
-</net>
+<junction x="127" y="-99.676"/>
+</segment>
+</net>

Commit message: Add files via upload
Parts:
- renumbered JP9 to MICRO_USB, U$1 to U11, U$2 to U10, U$5 to U12
Changed lines of the file:
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@@
 <part name="GND2" library="supply1" deviceset="GND" device=""/>
 <part name="GND13" library="supply1" deviceset="GND" device=""/>
-<part name="U$5" library="myLibraries" deviceset="SMF05C" device=""/>
+<part name="U12" library="myLibraries" deviceset="SMF05C" device=""/>
 <part name="GND14" library="supply1" deviceset="GND" device=""/>
 <part name="GND15" library="supply1" deviceset="GND" device=""/>
 <part name="GND12" library="supply1" deviceset="GND" device=""/>
-<part name="U$1" library="myLibraries" deviceset="MCP73831" device=""/>
+<part name="U11" library="myLibraries" deviceset="MCP73831" device=""/>
 <part name="R10" library="SparkFun-Resistors" deviceset="RESISTOR" device="0603-RES"/>
 <part name="R4" library="SparkFun-Resistors" deviceset="RESISTOR" device="0603-RES" value="470R"/>
@@
 <part name="C14" library="SparkFun-Capacitors" deviceset="CAP" device="0805" value="100nF"/>
 <part name="C15" library="SparkFun-Capacitors" deviceset="CAP" device="0805" value="33pF"/>
-<part name="U$2" library="myLibraries" deviceset="NANOSIM" device=""/>
 <part name="FRAME1" library="frames" deviceset="A3L-LOC" device=""/>
 <part name="D3" library="led" deviceset="LED" device="SML0603" value="GREEN (charged)"/>
-<part name="JP9" library="SparkFun-Connectors" deviceset="USB-AB" device="CONN-11794" value="Micro USB"/>
+<part name="MICRO_USB" library="SparkFun-Connectors" deviceset="USB-AB" device="CONN-11794" value="Micro USB"/>
 <part name="TX" library="SparkFun-Connectors" deviceset="M01" device="PTH"/>
 <part name="Q1" library="SparkFun-DiscreteSemi" deviceset="TRANSISTOR_NPN" device="MMBT2222A" value="MMBT2222A"/>
@@
 <part name="GND8" library="SparkFun-Aesthetics" deviceset="GND" device=""/>
 <part name="JP2" library="Various_parts" deviceset="TC2030-NL" device=""/>
+<part name="U10" library="myLibraries" deviceset="NANOSIM" device=""/>
 </parts>
 <sheets>
@@
 <instance part="GND2" gate="1" x="-185.42" y="-81.28"/>
 <instance part="GND13" gate="1" x="-81.28" y="-43.18"/>
-<instance part="U$5" gate="G$1" x="30.48" y="-71.12" rot="R90"/>
+<instance part="U12" gate="G$1" x="30.48" y="-71.12" rot="R90"/>
 <instance part="GND14" gate="1" x="38.1" y="22.86"/>
 <instance part="GND15" gate="1" x="33.02" y="40.64"/>
 <instance part="GND12" gate="1" x="15.24" y="58.42"/>
-<instance part="U$1" gate="G$1" x="-160.02" y="71.12"/>
+<instance part="U11" gate="G$1" x="-160.02" y="71.12"/>
 <instance part="R10" gate="G$1" x="-139.7" y="63.5" smashed="yes" rot="R90">
 <attribute name="NAME" x="-141.1986" y="59.69" size="1.778" layer="95" rot="R90"/>
@@
 </instance>
 <instance part="C15" gate="G$1" x="-68.58" y="-35.56"/>
-<instance part="U$2" gate="G$1" x="-22.86" y="-50.8" rot="MR0"/>
 <instance part="FRAME1" gate="G$1" x="-233.68" y="-147.32"/>
 <instance part="D3" gate="G$1" x="-185.42" y="60.96" smashed="yes">
@@
 <attribute name="VALUE" x="-192.532" y="52.705" size="1.778" layer="96"/>
 </instance>
-<instance part="JP9" gate="G$1" x="-215.9" y="66.04" smashed="yes" rot="R180"/>
+<instance part="MICRO_USB" gate="G$1" x="-215.9" y="66.04" smashed="yes" rot="R180"/>
 <instance part="TX" gate="G$1" x="116.84" y="58.42" rot="R180"/>
 <instance part="Q1" gate="G$1" x="-12.7" y="-116.84"/>
@@
 <instance part="GND8" gate="1" x="-96.52" y="55.88"/>
 <instance part="JP2" gate="G$1" x="83.82" y="5.08"/>
+<instance part="U10" gate="G$1" x="-22.86" y="-50.8" smashed="yes" rot="MR0">
+<attribute name="NAME" x="-21.082" y="-42.418" size="2.54" layer="95" rot="MR0"/>
+<attribute name="VALUE" x="-20.32" y="-60.96" size="1.27" layer="96" rot="MR0"/>
+</instance>
 </instances>
 <busses>
@@
 <pinref part="R10" gate="G$1" pin="1"/>
 <wire x1="-139.7" y1="58.42" x2="-139.7" y2="55.88" width="0.1524" layer="91"/>
-<pinref part="U$1" gate="G$1" pin="VSS"/>
+<pinref part="U11" gate="G$1" pin="VSS"/>
 <wire x1="-147.32" y1="66.04" x2="-147.32" y2="55.88" width="0.1524" layer="91"/>
 <pinref part="GND7" gate="1" pin="GND"/>
@@
 <pinref part="D3" gate="G$1" pin="C"/>
 <junction x="-185.42" y="55.88"/>
-<pinref part="JP9" gate="G$1" pin="GND"/>
+<pinref part="MICRO_USB" gate="G$1" pin="GND"/>
 <wire x1="-210.82" y1="60.96" x2="-210.82" y2="55.88" width="0.1524" layer="91"/>
 </segment>
@@
 </segment>
 <segment>
-<wire x1="-38.1" y1="-55.88" x2="-35.56" y2="-55.88" width="0.1524" layer="91"/>
 <pinref part="C5" gate="G$1" pin="2"/>
 <wire x1="-25.4" y1="-35.56" x2="-38.1" y2="-35.56" width="0.1524" layer="91"/>
 <wire x1="-38.1" y1="-35.56" x2="-38.1" y2="-55.88" width="0.1524" layer="91"/>
 <pinref part="GND3" gate="1" pin="GND"/>
+<pinref part="U10" gate="G$1" pin="GND"/>
+<wire x1="-35.56" y1="-55.88" x2="-38.1" y2="-55.88" width="0.1524" layer="91"/>
 <junction x="-38.1" y="-55.88"/>
-<pinref part="U$2" gate="G$1" pin="GND"/>
-</segment>
-<segment>
-<pinref part="U$5" gate="G$1" pin="2"/>
+</segment>
+<segment>
+<pinref part="U12" gate="G$1" pin="2"/>
 <pinref part="GND19" gate="1" pin="GND"/>
 </segment>
@@
 <wire x1="5.08" y1="-55.88" x2="15.24" y2="-55.88" width="0.1524" layer="91"/>
 <wire x1="15.24" y1="-55.88" x2="15.24" y2="-81.28" width="0.1524" layer="91"/>
-<pinref part="U$5" gate="G$1" pin="1"/>
+<pinref part="U12" gate="G$1" pin="1"/>
 <wire x1="15.24" y1="-81.28" x2="25.4" y2="-81.28" width="0.1524" layer="91"/>
 <label x="7.62" y="-55.88" size="1.778" layer="95"/>
@@
 <wire x1="5.08" y1="-50.8" x2="25.4" y2="-50.8" width="0.1524" layer="91"/>
 <label x="7.62" y="-50.8" size="1.778" layer="95"/>
-<pinref part="U$5" gate="G$1" pin="6"/>
+<pinref part="U12" gate="G$1" pin="6"/>
 <wire x1="25.4" y1="-60.96" x2="25.4" y2="-50.8" width="0.1524" layer="91"/>
 </segment>
@@
 <wire x1="-10.16" y1="-45.72" x2="30.48" y2="-45.72" width="0.1524" layer="91"/>
 <label x="7.62" y="-45.72" size="1.778" layer="95"/>
-<pinref part="U$5" gate="G$1" pin="5"/>
+<pinref part="U12" gate="G$1" pin="5"/>
 <wire x1="30.48" y1="-45.72" x2="30.48" y2="-60.96" width="0.1524" layer="91"/>
-<pinref part="U$2" gate="G$1" pin="VCC"/>
+<pinref part="U10" gate="G$1" pin="VCC"/>
 <junction x="-10.16" y="-45.72"/>
 </segment>
@@
 <net name="VBAT" class="0">
 <segment>
-<pinref part="U$1" gate="G$1" pin="VBAT"/>
+<pinref part="U11" gate="G$1" pin="VBAT"/>
 <wire x1="-147.32" y1="76.2" x2="-132.08" y2="76.2" width="0.1524" layer="91"/>
 <wire x1="-132.08" y1="71.12" x2="-132.08" y2="76.2" width="0.1524" layer="91"/>
@@
 </segment>
 </net>
-<net name="N$7" class="0">
-<segment>
-<wire x1="-10.16" y1="-50.8" x2="-5.08" y2="-50.8" width="0.1524" layer="91"/>
-<pinref part="R1" gate="G$1" pin="1"/>
-<pinref part="U$2" gate="G$1" pin="RST"/>
-</segment>
-</net>
 <net name="N$18" class="0">
 <segment>
 <pinref part="D2" gate="G$1" pin="A"/>
-<pinref part="JP9" gate="G$1" pin="VBUS"/>
+<pinref part="MICRO_USB" gate="G$1" pin="VBUS"/>
 <wire x1="-208.28" y1="76.2" x2="-210.82" y2="76.2" width="0.1524" layer="91"/>
 <wire x1="-210.82" y1="76.2" x2="-210.82" y2="71.12" width="0.1524" layer="91"/>
@@
 <net name="N$16" class="0">
 <segment>
-<pinref part="U$1" gate="G$1" pin="PROG"/>
+<pinref part="U11" gate="G$1" pin="PROG"/>
 <wire x1="-147.32" y1="71.12" x2="-139.7" y2="71.12" width="0.1524" layer="91"/>
 <wire x1="-139.7" y1="71.12" x2="-139.7" y2="68.58" width="0.1524" layer="91"/>
@@
 <net name="N$22" class="0">
 <segment>
-<pinref part="U$1" gate="G$1" pin="VDD"/>
+<pinref part="U11" gate="G$1" pin="VDD"/>
 <wire x1="-198.12" y1="76.2" x2="-185.42" y2="76.2" width="0.1524" layer="91"/>
 <wire x1="-185.42" y1="76.2" x2="-172.72" y2="76.2" width="0.1524" layer="91"/>
@@
 <net name="N$14" class="0">
 <segment>
-<pinref part="U$1" gate="G$1" pin="STAT"/>
+<pinref part="U11" gate="G$1" pin="STAT"/>
 <pinref part="R4" gate="G$1" pin="1"/>
 <wire x1="-175.26" y1="66.04" x2="-172.72" y2="66.04" width="0.1524" layer="91"/>
@@
 </segment>
 </net>
-<net name="N$3" class="0">
-<segment>
-<wire x1="-5.08" y1="-55.88" x2="-10.16" y2="-55.88" width="0.1524" layer="91"/>
-<pinref part="R5" gate="G$1" pin="1"/>
-<pinref part="U$2" gate="G$1" pin="CLK"/>
-</segment>
-</net>
 <net name="RESET" class="0">
 <segment>
@@
 <pinref part="R7" gate="G$1" pin="1"/>
 <wire x1="-43.18" y1="-50.8" x2="-45.828" y2="-50.8" width="0.1524" layer="91"/>
-<wire x1="-43.18" y1="-45.72" x2="-43.18" y2="-50.8" width="0.1524" layer="91"/>
-<wire x1="-35.56" y1="-45.72" x2="-43.18" y2="-45.72" width="0.1524" layer="91"/>
+<wire x1="-43.18" y1="-50.8" x2="-43.18" y2="-45.72" width="0.1524" layer="91"/>
+<pinref part="U12" gate="G$1" pin="4"/>
 <wire x1="-43.18" y1="-45.72" x2="-43.18" y2="-25.4" width="0.1524" layer="91"/>
-<pinref part="U$5" gate="G$1" pin="4"/>
 <wire x1="-43.18" y1="-25.4" x2="35.56" y2="-25.4" width="0.1524" layer="91"/>
 <wire x1="35.56" y1="-25.4" x2="35.56" y2="-60.96" width="0.1524" layer="91"/>
+<pinref part="U10" gate="G$1" pin="I/O"/>
+<wire x1="-35.56" y1="-45.72" x2="-43.18" y2="-45.72" width="0.1524" layer="91"/>
 <junction x="-43.18" y="-45.72"/>
-<pinref part="U$2" gate="G$1" pin="I/O"/>
 </segment>
 </net>
@@
 </segment>
 </net>
+<net name="N$3" class="0">
+<segment>
+<pinref part="R1" gate="G$1" pin="1"/>
+<pinref part="U10" gate="G$1" pin="RST"/>
+<wire x1="-5.08" y1="-50.8" x2="-10.16" y2="-50.8" width="0.1524" layer="91"/>
+</segment>
+</net>
+<net name="N$7" class="0">
+<segment>
+<pinref part="R5" gate="G$1" pin="1"/>
+<pinref part="U10" gate="G$1" pin="CLK"/>
+<wire x1="-5.08" y1="-55.88" x2="-10.16" y2="-55.88" width="0.1524" layer="91"/>
+</segment>
+</net>

Commit message: Add files via upload
Parts:
- C14, C15: device SparkFun-Capacitors:CAP0805 -> SparkFun-Capacitors:CAP0603-CAP
- R10: value (none) -> 2K
Other:
- moved on the sheet: C14, C15
Changed lines of the file:
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@@
 <part name="GND12" library="supply1" deviceset="GND" device=""/>
 <part name="U11" library="myLibraries" deviceset="MCP73831" device=""/>
-<part name="R10" library="SparkFun-Resistors" deviceset="RESISTOR" device="0603-RES"/>
+<part name="R10" library="SparkFun-Resistors" deviceset="RESISTOR" device="0603-RES" value="2K"/>
 <part name="R4" library="SparkFun-Resistors" deviceset="RESISTOR" device="0603-RES" value="470R"/>
 <part name="D1" library="led" deviceset="LED" device="SML0603" value="RED (charging)"/>
@@
 <part name="U1" library="SparkFun-DigitalIC" deviceset="ATMEGA328P_TQFP" device="" value="ATMEGA328P_TQFP"/>
 <part name="C6" library="SparkFun-Capacitors" deviceset="CAP" device="1206" value="100uF/6.3V"/>
-<part name="C14" library="SparkFun-Capacitors" deviceset="CAP" device="0805" value="100nF"/>
-<part name="C15" library="SparkFun-Capacitors" deviceset="CAP" device="0805" value="33pF"/>
 <part name="FRAME1" library="frames" deviceset="A3L-LOC" device=""/>
 <part name="D3" library="led" deviceset="LED" device="SML0603" value="GREEN (charged)"/>
@@
 <part name="JP2" library="Various_parts" deviceset="TC2030-NL" device=""/>
 <part name="U10" library="myLibraries" deviceset="NANOSIM" device=""/>
+<part name="C15" library="SparkFun-Capacitors" deviceset="CAP" device="0603-CAP" value="33pF"/>
+<part name="C14" library="SparkFun-Capacitors" deviceset="CAP" device="0603-CAP" value="100nF"/>
 </parts>
 <sheets>
@@
 <attribute name="VALUE" x="-94.361" y="-39.116" size="1.778" layer="96" rot="R90"/>
 </instance>
-<instance part="C14" gate="G$1" x="-81.28" y="-35.56" smashed="yes">
-<attribute name="NAME" x="-79.756" y="-32.639" size="1.778" layer="95"/>
-<attribute name="VALUE" x="-79.756" y="-37.719" size="1.778" layer="96"/>
-</instance>
-<instance part="C15" gate="G$1" x="-68.58" y="-35.56"/>
 <instance part="FRAME1" gate="G$1" x="-233.68" y="-147.32"/>
 <instance part="D3" gate="G$1" x="-185.42" y="60.96" smashed="yes">
@@
 <attribute name="VALUE" x="-20.32" y="-60.96" size="1.27" layer="96" rot="MR0"/>
 </instance>
+<instance part="C15" gate="G$1" x="-68.58" y="-33.938"/>
+<instance part="C14" gate="G$1" x="-81.28" y="-33.938"/>
 </instances>
 <busses>
@@
 <wire x1="-91.44" y1="-38.1" x2="-91.44" y2="-40.64" width="0.1524" layer="91"/>
 <wire x1="-91.44" y1="-40.64" x2="-81.28" y2="-40.64" width="0.1524" layer="91"/>
-<pinref part="C15" gate="G$1" pin="2"/>
 <wire x1="-81.28" y1="-40.64" x2="-68.58" y2="-40.64" width="0.1524" layer="91"/>
-<wire x1="-68.58" y1="-40.64" x2="-68.58" y2="-38.1" width="0.1524" layer="91"/>
-<pinref part="C14" gate="G$1" pin="2"/>
-<wire x1="-81.28" y1="-38.1" x2="-81.28" y2="-40.64" width="0.1524" layer="91"/>
+<wire x1="-68.58" y1="-40.64" x2="-68.58" y2="-36.478" width="0.1524" layer="91"/>
+<wire x1="-68.58" y1="-36.478" x2="-68.58" y2="-38.1" width="0.1524" layer="91"/>
+<wire x1="-81.28" y1="-38.1" x2="-81.28" y2="-36.478" width="0.1524" layer="91"/>
 <pinref part="GND13" gate="1" pin="GND"/>
 <junction x="-81.28" y="-40.64"/>
+<pinref part="C15" gate="G$1" pin="2"/>
+<junction x="-68.58" y="-36.478"/>
+<pinref part="C14" gate="G$1" pin="2"/>
+<wire x1="-81.28" y1="-36.478" x2="-81.28" y2="-40.64" width="0.1524" layer="91"/>
+<junction x="-81.28" y="-36.478"/>
 </segment>
 <segment>
@@
 <pinref part="C6" gate="G$1" pin="1"/>
 <wire x1="-91.44" y1="-30.48" x2="-91.44" y2="-25.4" width="0.1524" layer="91"/>
-<pinref part="C15" gate="G$1" pin="1"/>
 <wire x1="-91.44" y1="-25.4" x2="-81.28" y2="-25.4" width="0.1524" layer="91"/>
 <wire x1="-81.28" y1="-25.4" x2="-68.58" y2="-25.4" width="0.1524" layer="91"/>
-<wire x1="-68.58" y1="-25.4" x2="-68.58" y2="-30.48" width="0.1524" layer="91"/>
-<pinref part="C14" gate="G$1" pin="1"/>
-<wire x1="-81.28" y1="-30.48" x2="-81.28" y2="-25.4" width="0.1524" layer="91"/>
+<wire x1="-68.58" y1="-25.4" x2="-68.58" y2="-28.858" width="0.1524" layer="91"/>
+<wire x1="-68.58" y1="-28.858" x2="-68.58" y2="-30.48" width="0.1524" layer="91"/>
+<wire x1="-81.28" y1="-30.48" x2="-81.28" y2="-28.858" width="0.1524" layer="91"/>
 <junction x="-81.28" y="-25.4"/>
 <label x="-78.74" y="-25.4" size="1.778" layer="95"/>
-</segment>
-<segment>
+<pinref part="C14" gate="G$1" pin="1"/>
+<wire x1="-81.28" y1="-28.858" x2="-81.28" y2="-25.4" width="0.1524" layer="91"/>
+<junction x="-81.28" y="-28.858"/>
+<pinref part="C15" gate="G$1" pin="1"/>
+<junction x="-68.58" y="-28.858"/>
+</segment>
+<segment>
